File: schematics/v5/shield_v5.sch (EAGLE design)
At the start: 47 parts, among them IC1 L293DD, IC2 74HCT04D, Q2 PMV20EN, Q3 PMV20EN, Q4 PMV20EN, Q5 PMV20EN, U1 ATMEGA168

Commit message: cleaned schematics
Parts:
- removed R2: (no value), rcl:R-EU_M1206
- added C12: (no value), rcl:C-EUC1206
Connections:
- net N$10 renamed PB0
- net N$13 renamed PD2
- net N$15 renamed PC1
- net N$16 renamed PC2
- net N$17 renamed PC3
- net N$2 renamed UNCONNECTED_GND
- net N$4 renamed PD7
- new net D0: SV3.5
- net N$9: now also C12.2; no longer R2.2
- net RESET: now also C12.1; no longer R2.1
Other:
- note added: "ADC in / Digital In/Out"
- note added: "Accel connector"
- note added: "Controller"
- note added: "Digital In/Out, Ws2812"
- note added: "Direct CHIP In/Output"
- note added: "IN-/OUTPUTs"
- note added: "LED section"
- note added: "Left connector"
- note added: "Lower GND (out)"
- note added: "Motor section"
- note added: "PWM(to GND) / Motor"
- note added: "PWM, Ws2812, Digital"
- note added: "Pad10"
- note added: "Pad11"
- note added: "Pad12"
- note added: "Pin0"
- note added: "Pin1"
- note added: "Pin2"
- note added: "Pin3"
- note added: "Pin4"
- note added: "Pin5"
- note added: "Pin6"
- note added: "Pin7"
- note added: "Pin8"
- note added: "Pin9"
- note added: "Power selection"
- note added: "Right connector"
- note added: "UART connector"
- note added: "Upper GND (in)"
- note added: "Vin (upper)"
- note added: "Vout (lower)"
- moved on the sheet: C1, C2, C3, C4, IC1, IC2A, IC2B, IC2P, JP2, JP3, JP4, LED2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
