File: schematics/v7/shield_v7.brd (EAGLE design)
At the start: 41 x 50 mm, 51 parts, among them IC1 L293DD, IC2 74HCT04D, Q2 PMV20EN, Q3 PMV20EN, Q4 PMV20EN, Q5 PMV20EN, U1 ATMEGA168

Commit message: moved motor driver lower
Parts:
- moved C3 10.9 mm to (33.8, 37.4), turned to 90 degrees
- moved U$2 6.99 mm to (23.8, 19.3)
- moved IC1 1.27 mm to (16.0, 33.9)
- moved C2 1.00 mm to (7.78, 27.3)
- moved IC2 0.76 mm to (28.3, 37.1)
Routing:
- net GND: track 279.4 -> 253.4 mm, vias 8 -> 9
- net VCC: track 109.9 -> 102.8 mm
- net P1: track 22.7 -> 20.1 mm
- net PO4: track 25.8 -> 28.2 mm
- net IN1: track 38.9 -> 36.7 mm
- net N$11: track 7.24 -> 5.42 mm
- net OC1_PWM2: track 47.4 -> 45.7 mm
- net IN3: track 48.7 -> 47.0 mm
- net N$1: track 40.4 -> 38.7 mm
- net VIN: track 31.6 -> 32.8 mm
- net PO1: track 19.3 -> 20.6 mm
- net PC3: track 16.5 -> 17.6 mm
Other:
- board text added: "10"
- board text added: "11"
- board text added: "12"
- board text added: "8: A_IN"
- board text added: "9"
- board text added: "C.H.I.P. SALSA DIP v2.5 JKW"
- board text removed: "SALSA DIP v2.5 C.H.I.P. JKW"
