File: schematics/v9/shield_v9.brd (EAGLE design)
At the start: 41 x 50 mm, 54 parts, among them IC1 L293DD, IC2 74HCT04D, Q2 PMV20EN, Q3 PMV20EN, Q4 PMV20EN, Q5 PMV20EN, U1 ATMEGA168

Commit message: added gerber files for ordered version
Parts:
- C12: value (none) -> 100nF
Changed lines of the file:
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@@
 <attribute name="VALUE" x="30" y="12.23" size="0.0254" layer="27" rot="R90"/>
 </element>
-<element name="C12" library="rcl" package="C1206" value="" x="9.04" y="6.73" smashed="yes" rot="MR0">
+<element name="C12" library="rcl" package="C1206" value="100nF" x="9.04" y="6.73" smashed="yes" rot="MR0">
 <attribute name="VALUE" x="10.31" y="4.19" size="1.27" layer="28" rot="MR0"/>
 </element>
