File: schematics/dev_versions/Salsa_II_v3.9/shield_v9.brd (EAGLE design)
At the start: 41 x 50 mm, 52 parts, among them IC1 L293DD, IC2 74HCT04D, Q2 PMV20EN, Q3 PMV20EN, Q4 PMV20EN, Q5 PMV20EN, U1 ATMEGA168

Commit message: cleaned version structure for forum
Parts:
- removed PAD13: (no value), wirepad:SMD1,27-2,54
- removed PAD14, PAD16, PAD18: (no value), wirepad:3,17/1,3
- added PAD0, PAD_G1, PAD_G2, PAD_VIN: (no value), wirepad:3,17/1,3
- added S1: SMD-1101NE, SparkFun-Electromechanical:TACTILE-SWITCH-1101NE
- added SJA, SJO: (no value), jumper:SJ
- C4: value (none) -> 10u
- PAD11: value (none) -> WIREPADSMD1,27-254; device wirepad:3,17/1,3 -> wirepad:SMD1,27-2,54
- PAD8: value WIREPADSMD1,27-254 -> (none); device wirepad:SMD1,27-2,54 -> wirepad:3,17/1,3
- PAD9: device wirepad:3,17/1,3 -> wirepad:SMD1,27-2,54
- SJC4: value (none) -> SJC4
- moved PAD4 44.3 mm to (13.0, 3.00)
- moved PAD5 44.3 mm to (18.0, 3.00)
- moved PAD6 44.3 mm to (23.0, 3.00)
- moved PAD10 30.1 mm to (32.8, 9.18)
- moved PAD11 23.8 mm to (24.4, 31.5), flipped to the bottom, turned to 180 degrees
- moved PAD9 18.8 mm to (29.6, 11.9), turned to 180 degrees
- moved PAD8 17.8 mm to (7.58, 25.6), flipped to the top, turned to 0 degrees
- moved PAD1 15.0 mm to (18.0, 47.0)
- moved PAD2 15.0 mm to (23.0, 47.0)
- moved PAD3 15.0 mm to (28.0, 47.0)
- moved LED2 7.09 mm to (10.5, 19.2), turned to 180 degrees
- moved PAD7 5.00 mm to (28.0, 3.00)
- moved R4 2.46 mm to (15.4, 14.4), turned to 0 degrees
- moved C4 0.69 mm to (9.32, 32.2)
- moved D3 0.44 mm to (9.37, 36.0)
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- renumbered SJ6 to SJC4, SJ7 to SJC3, SJ8 to SJC, SJ9 to SJC2
Connections:
- removed net N$26: LED2.A, U1.23
- removed net N$7: D1.A, U$1.VOUT
- new net EN1: IC1.1, SJA.1, SJC.1, SJO.1
- new net PC0: S1.P$2, U1.23
- new net VREG: D1.A, SV2.36, U$1.VOUT
- net GND: now also PAD_G1.1, PAD_G2.1, S1.P$1, SJO.2; no longer PAD1.1, PAD7.1
- net INT1: now also PAD5.1; no longer PAD16.1
- net OC2_PWM1: now also PAD9.1, SJA.2; no longer IC1.1, PAD13.1, SJC.1
- net OC2_PWM2: now also LED2.A, PAD7.1; no longer PAD18.1
- net P3: now also SJC.2
- net P4: no longer SJC.2
- net PB0: now also PAD11.1; no longer PAD8.1
- net PC1: now also PAD4.1; no longer PAD9.1
- net PC2: now also PAD8.1; no longer PAD10.1
- net PC3: now also PAD10.1; no longer PAD11.1
- net PD2: now also PAD6.1; no longer PAD14.1
- net PO1: now also PAD0.1; no longer PAD3.1
- net PO2: now also PAD1.1; no longer PAD4.1
- net PO3: now also PAD2.1; no longer PAD5.1
- net PO4: now also PAD3.1; no longer PAD6.1
- net VCC: no longer SV2.36
- net VIN_SCREW: now also PAD_VIN.1; no longer PAD2.1
Routing:
- net VREG: track 0.00 -> 55.1 mm, vias 0 -> 2
- net P3: track 0.00 -> 22.9 mm, vias 0 -> 1
- net P4: track 20.0 -> 0.00 mm, vias 1 -> 0
- net GND: track 278.2 -> 295.7 mm, vias 11 -> 12
- net IN1: track 25.6 -> 36.5 mm
- net EN1: track 0.00 -> 9.45 mm, vias 0 -> 1
- net N$7: track 6.96 -> 0.00 mm
- net VCC: track 136.3 -> 129.7 mm, vias 7 -> 9
- net OC2_PWM1: track 32.2 -> 26.5 mm, vias 2 -> 1
- net OC2_PWM2: track 45.4 -> 49.7 mm
- net N$26: track 3.84 -> 0.00 mm
- net PD2: track 16.1 -> 12.5 mm
- net SDA: track 47.0 -> 50.0 mm
- net PC0: track 0.00 -> 2.60 mm
- net N$4: track 3.83 -> 6.10 mm
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- added copper zone on layer 1, net VCC
- added copper zone on layer 1, net VIN_SCREW
Other:
- board text added: "JKW v3.a"
- board text added: "SALSA DIP II v3.a"
- board text removed: "SALSA DIP v3.9"
