File: schematics/dev_versions/Salsa_II_v3.9/shield_v9.sch (EAGLE design)
At the start: 50 parts, among them IC1 L293DD, IC2 74HCT04D, Q2 PMV20EN, Q3 PMV20EN, Q4 PMV20EN, Q5 PMV20EN, U1 ATMEGA168

Commit message: cleaned version structure for forum
Parts:
- removed PAD13: (no value), wirepad:SMD2
- removed PAD14, PAD16, PAD18: (no value), wirepad:3,17/1,3
- removed SJ8: (no value), jumper:SJ
- added PAD0, PAD_G1, PAD_G2, PAD_VIN: (no value), wirepad:3,17/1,3
- added S1: SMD-1101NE, SparkFun-Electromechanical:SWITCH-MOMENTARY-2-SMD-1101NE
- added SJA, SJC, SJO: (no value), jumper:SJ
- C4: value (none) -> 10u
- PAD11: value (none) -> WIREPADSMD1,27-254; device wirepad:3,17/1,3 -> wirepad:WIREPADSMD1,27-254
- PAD8: value WIREPADSMD1,27-254 -> (none); device wirepad:WIREPADSMD1,27-254 -> wirepad:3,17/1,3
- PAD9: device wirepad:3,17/1,3 -> wirepad:SMD2
- SJC4: value (none) -> SJC4
- renumbered SJ6 to SJC4, SJ7 to SJC3, SJ9 to SJC2
Connections:
- removed net N$26: LED2.A, U1.PC0(ADC0)
- removed net N$7: D1.A, U$1.VOUT
- new net EN1: IC1.EN1, SJA.1, SJC.1, SJO.1
- new net PC0: S1.2, U1.PC0(ADC0)
- new net VREG: D1.A, SV2.36, U$1.VOUT
- net GND: now also PAD_G1.P, PAD_G2.P, S1.1, SJO.2; no longer PAD1.P, PAD7.P
- net INT1: now also PAD5.P; no longer PAD16.P
- net OC2_PWM1: now also PAD9.P, SJA.2; no longer IC1.EN1, PAD13.P, SJ8.1
- net OC2_PWM2: now also LED2.A, PAD7.P; no longer PAD18.P
- net P3: now also SJC.2
- net P4: no longer SJ8.2
- net PB0: now also PAD11.P; no longer PAD8.P
- net PC1: now also PAD4.P; no longer PAD9.P
- net PC2: now also PAD8.P; no longer PAD10.P
- net PC3: now also PAD10.P; no longer PAD11.P
- net PD2: now also PAD6.P; no longer PAD14.P
- net PO1: now also PAD0.P; no longer PAD3.P
- net PO2: now also PAD1.P; no longer PAD4.P
- net PO3: now also PAD2.P; no longer PAD5.P
- net PO4: now also PAD3.P; no longer PAD6.P
- net VCC: no longer SV2.36
- net VIN_SCREW: now also PAD_VIN.P; no longer PAD2.P
Other:
- note added: "3.0V (>1.8V)"
- note added: "3.7V"
- note added: "4.3V (>1.8V)"
- note added: "4.8V! (>1.8V)"
- note added: "5.0V"
- note added: "5.5V!"
- note added: "If SJC, SJC2, SJC3, SJC4 are set avoid using the Atmega pins"
- note added: "One out of Ws2812 or LED or switch"
- note added: "Only set SJC or SJA or SJ0 If SJC is set, CHIP is controlling the Driver SJA = Atmega in controll SJ0 = OUT1/2 are disabled"
- note added: "Pad9"
- note added: "Pin10"
- note removed: "Pad10"
- note removed: "Pin9"
- moved on the sheet: C2, C5, D1, LED2, PAD1, PAD10, PAD12, PAD3, PAD4, PAD5, PAD6, PAD7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
